Commit message: add normalcam

File: diff_robot_description/urdf/diff_robot.materials.xacro (robot description, xacro)
@@ -2,10 +2,10 @@
 <robot xmlns:xacro="http://www.ros.org/wiki/xacro">
     <!--__________Material__________-->
-    <material name="yellow">
+  <!-- <material name="yellow">
         <color rgba="0.8 0.3 0.1 0.5" />
-    </material>
-    <material name="black">
+    </material> -->
+    <!-- <material name="black">
         <color rgba="0.0 0.0 0.0 1.0" />
-    </material>
+    </material> -->
     <material name="blue">
         <color rgba="0 0 0.5 1" />

File: diff_robot_description/urdf/diff_robot.urdf.xacro (robot description, xacro)
@@ -1,5 +1,5 @@
 <?xml version="1.0"?>
 <robot xmlns:xacro="http://www.ros.org/wiki/xacro" name="diff_robot">
-  <xacro:include filename="$(find diff_robot_description)/urdf/diff_robot.materials.xacro" />
+  <!-- <xacro:include filename="$(find diff_robot_description)/urdf/diff_robot.materials.xacro" /> -->
   <xacro:include filename="$(find diff_robot_description)/urdf/diff_robot_description.urdf.xacro" />
 </robot>
